File: Documents/KiCad/ardPowerTempLog no peripherals unrouted.kicad_pcb (KiCad board)
At the start: 2 copper layers, 36 parts, among them J1 R1, J10 5-pin_3-pole_3,5mm_audio_head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, J11 4-pin_3LED_header, J12 Conn_01x02_Male, J13 Conn_01x02_Male, J2 S2, J3 T3, J4 OneWire bus, J5 LED sensor, J6 5-pin_3-pole_3,5mm_audio_head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

Commit message: kicad
Parts:
- removed D1: Status LED, LED_THT:LED_D5.0mm
- removed D2: Polled LED, LED_THT:LED_D5.0mm
- removed D3: Pulse LED, LED_THT:LED_D5.0mm
- removed J1: R1, My_Misc:My_Jack_3.5mm_Ledino_KB3SPRS_Horizontal
- removed J2: S2, My_Misc:My_Jack_3.5mm_Ledino_KB3SPRS_Horizontal
- removed J3: T3, My_Misc:My_Jack_3.5mm_Ledino_KB3SPRS_Horizontal
- removed J4: OneWire bus, My_Misc:My_Jack_3.5mm_Ledino_KB3SPRS_Horizontal
- removed J5: LED sensor, My_Misc:My_Jack_3.5mm_Ledino_KB3SPRS_Horizontal
- removed Q1: Q_Photo_NPN_CBE, Package_TO_SOT_THT:TO-18-3
- removed U1: DS18B20, Package_TO_SOT_THT:TO-92_Inline
- moved R11 12.8 mm to (133.3, 97.8)
- moved R12 12.7 mm to (154.9, 97.8)
- moved R1 6.39 mm to (133.3, 91.4)
- moved R5 6.39 mm to (133.3, 85.1)
- moved R2 6.35 mm to (154.9, 91.4)
- moved R6 6.35 mm to (154.9, 85.1)
- moved C1 2.84 mm to (148.6, 88.9), turned to 90 degrees
- moved C2 1.27 mm to (170.2, 88.9), turned to 90 degrees
