File: Documents/KiCad/ardPowerTempLog no peripherals routed1 gnd copper pour.kicad_pcb (KiCad board)
At the start: 2 copper layers, 68.6 x 53.3 mm, 26 parts, among them J10 5-pin_3-pole_3,5mm_audio_head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, J11 4-pin_3LED_header, J12 Conn_01x02_Male, J13 Conn_01x02_Male, J6 5-pin_3-pole_3,5mm_audio_head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, J7 5-pin_3-pole_3,5mm_audio_head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, J8 5-pin_3-pole_3,5mm_audio_head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, J9 5-pin_3-pole_3,5mm_audio_head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

Commit message: schematics
Parts:
- moved J11 20.4 mm to (144.8, 66.0)
- moved R15 15.2 mm to (166.4, 66.0), turned to 270 degrees
- moved R17 13.0 mm to (153.7, 66.0), turned to 270 degrees
- moved R16 10.9 mm to (160.0, 66.0), turned to 270 degrees
- moved J9 10.2 mm to (109.2, 77.5)
- moved R13 5.08 mm to (109.2, 68.6)
Routing:
- net /GND: track 0.00 -> 208.0 mm, vias 0 -> 2
- net /Collector: track 0.00 -> 117.6 mm, vias 0 -> 4
- net /Data: track 0.00 -> 68.3 mm
- net Net-(A1-Pad19): track 0.00 -> 60.0 mm
- net Net-(A1-Pad10): track 0.00 -> 58.3 mm
- net Net-(A1-Pad11): track 0.00 -> 36.7 mm
- net Net-(C2-Pad1): track 0.00 -> 36.4 mm
- net Net-(C3-Pad1): track 0.00 -> 36.4 mm
- net Net-(C1-Pad1): track 0.00 -> 36.4 mm
- net Net-(D1-Pad2): track 0.00 -> 25.8 mm
- net Net-(A1-Pad12): track 0.00 -> 19.1 mm
- net /Emitter: track 0.00 -> 19.0 mm
- net Net-(D2-Pad2): track 0.00 -> 18.4 mm
- net Net-(A1-Pad22): track 0.00 -> 17.3 mm
- net Net-(A1-Pad23): track 0.00 -> 15.1 mm
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- added copper zone on B.Cu, net /GND
Other:
- board text added: "5V"
- board text added: "GND"
- board text removed: "D4"
