File: piHeating/Documents/KiCad/piHeatingRPi1.kicad_pcb (KiCad board)
At the start: 2 copper layers, 62.2 x 50.8 mm, 17 parts, among them J1 Raspberry_Pi_1_all_pin_ordered, J2 10-pin_header_LCD_interface, J3 3-pin_KY-019_relay_header, J4 3_pin_Dallas_1-wire_connector, J5 2-pin_NO_switch_header, J6 2-pin_NO_switch_header, J7 2-pin_NO_switch_header, J8 2-pin_NO_switch_header

Commit message: kicad for rpi1
Parts:
- moved J1 1.87 mm to (176.5, 46.1)
Routing:
- net Net-(J1-Pad1): track 68.0 -> 75.7 mm
- net Net-(J1-Pad2): track 43.7 -> 51.3 mm
- net Net-(J1-Pad10): track 53.6 -> 58.7 mm
- net Net-(J1-Pad18): track 104.9 -> 109.0 mm
- net Net-(J1-Pad8): track 37.4 -> 41.3 mm
- net Net-(J1-Pad12): track 55.8 -> 59.8 mm
- net Net-(J1-Pad16): track 80.5 -> 84.4 mm
- net Net-(J1-Pad22): track 130.0 -> 133.7 mm
- net Net-(J1-Pad25): track 97.8 -> 99.9 mm
- net Net-(J1-Pad11): track 10.8 -> 12.5 mm
- net Net-(J1-Pad15): track 10.8 -> 12.4 mm
- net Net-(J1-Pad19): track 13.3 -> 14.8 mm
- net Net-(J1-Pad13): track 11.0 -> 12.5 mm
- net Net-(J1-Pad7): track 11.3 -> 12.5 mm
- net Net-(J1-Pad21): track 13.4 -> 14.6 mm
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Other:
- board size 62.2 x 50.8 mm -> 64.8 x 50.8 mm

Commit message: better cad
Parts:
- moved R1 0.51 mm to (155.4, 57.1)
Routing:
- net Net-(J1-Pad2): track 51.3 -> 47.7 mm
- net Net-(J1-Pad1): track 75.7 -> 78.4 mm
- net Net-(J1-Pad10): track 58.7 -> 57.4 mm
- net Net-(J1-Pad7): track 12.5 -> 13.9 mm
- net Net-(J1-Pad25): track 99.9 -> 98.9 mm
- net Net-(J1-Pad8): track 41.3 -> 40.4 mm
Other:
- outline, holes or cut-outs redrawn
- net class 30: via_dia 2.032 -> 3.048
