File: piWeatherLog/Documents/KiCad/ardWeatherStation.kicad_pcb (KiCad board)
At the start: 2 copper layers, 12 parts, among them J1 RJ45, J2 RJ45, J3 10-pin_header_LCD_interface, U1 Rain_bucket, U2 Anemometer, U3 Wind_vane

Commit message: kicad, PCB
Parts:
- moved R1 32.8 mm to (142.2, 95.9)
- moved R3 29.0 mm to (142.2, 81.3)
- moved R2 28.3 mm to (142.2, 88.3)
- moved R4 19.9 mm to (152.4, 102.9), turned to 180 degrees
Routing:
- net Net-(A1-Pad20): track 0.00 -> 112.2 mm
- net Net-(A1-Pad11): track 0.00 -> 68.8 mm
- net Net-(A1-Pad29): track 0.00 -> 51.9 mm
- net Net-(A1-Pad5): track 0.00 -> 47.4 mm, vias 0 -> 2
- net Net-(A1-Pad19): track 0.00 -> 39.5 mm, vias 0 -> 2
- net Net-(D1-Pad1): track 0.00 -> 32.4 mm
- net (no net): track 0.00 -> 16.6 mm
- net Net-(A1-Pad28): track 0.00 -> 8.99 mm
- net Net-(A1-Pad27): track 0.00 -> 8.99 mm
- net Net-(A1-Pad26): track 0.00 -> 8.99 mm
- net Net-(A1-Pad25): track 0.00 -> 8.99 mm
- net Net-(A1-Pad24): track 0.00 -> 8.99 mm
- net Net-(A1-Pad23): track 0.00 -> 8.99 mm
- net Net-(A1-Pad17): track 0.00 -> 8.89 mm
- added copper zone on B.Cu, net (none)
- added copper zone on B.Cu, net Net-(A1-Pad29)
Other:
- board outline added: 69.8 x 54 mm
- net class 30 added: clearance 0.381, trace_width 0.762, via_dia 3.048, via_drill 0.4
- board text added: "5V"
- board text added: "D4"
- board text added: "R1"
- board text added: "R2"
- board text added: "R3"
- board text added: "R4"
- board text added: "ardWeatherStation Design: Jon Sagebrand jonsagebrand@gmail.com"
