File: KiCad/ardPowerTempLog/ardPowerTempLog.kicad_sch (KiCad schematic)
At the start: 35 parts, among them J1 R1, J10 5-pin_3-pole_3,5mm_audio_head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, J11 4-pin_3LED_header, J2 S2, J3 T3, J4 OneWire bus, J5 LED sensor, J6 5-pin_3-pole_3,5mm_audio_head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, J7 5-pin_3-pole_3,5mm_audio_head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, J8 5-pin_3-pole_3,5mm_audio_head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

Commit message: schematics
Parts:
- A1: footprint My_Arduino:Arduino_UNO_R3_shield_large -> Module:Arduino_UNO_R3
- J10, J6, J7, J8, J9: footprint (none) -> My_Headers:5-pin_3,5mm_audio_jack_header
- J11: footprint (none) -> My_Headers:4-pin_3_LED_header
- U1: footprint (none) -> Package_TO_SOT_THT:TO-92_Inline
Changed lines of the file:
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@@
     (property "Reference" "A1" (id 0) (at 147.32 50.0126 0))
     (property "Value" "Arduino_UNO_R3" (id 1) (at 147.32 52.324 0))
-    (property "Footprint" "My_Arduino:Arduino_UNO_R3_shield_large" (id 2) (at 147.32 80.01 0)
+    (property "Footprint" "Module:Arduino_UNO_R3" (id 2) (at 147.32 80.01 0)
       (effects (font (size 1.27 1.27) italic) hide)
     )
@@
       (effects (font (size 1.27 1.27)) (justify right))
     )
-    (property "Footprint" "" (id 2) (at 80.01 190.5 0)
+    (property "Footprint" "Package_TO_SOT_THT:TO-92_Inline" (id 2) (at 80.01 190.5 0)
       (effects (font (size 1.27 1.27)) hide)
     )
@@
       (effects (font (size 1.27 1.27)) hide)
     )
-    (property "Footprint" "" (id 2) (at 7.62 53.34 0)
+    (property "Footprint" "My_Headers:5-pin_3,5mm_audio_jack_header" (id 2) (at 7.62 53.34 0)
       (effects (font (size 1.27 1.27)) hide)
     )
@@
       (effects (font (size 1.27 1.27)) hide)
     )
-    (property "Footprint" "" (id 2) (at 7.62 100.33 0)
+    (property "Footprint" "My_Headers:5-pin_3,5mm_audio_jack_header" (id 2) (at 7.62 100.33 0)
       (effects (font (size 1.27 1.27)) hide)
     )
@@
       (effects (font (size 1.27 1.27)) hide)
     )
-    (property "Footprint" "" (id 2) (at 7.62 154.94 0)
+    (property "Footprint" "My_Headers:5-pin_3,5mm_audio_jack_header" (id 2) (at 7.62 154.94 0)
       (effects (font (size 1.27 1.27)) hide)
     )
@@
       (effects (font (size 1.27 1.27)) hide)
     )
-    (property "Footprint" "" (id 2) (at 287.02 46.99 0)
+    (property "Footprint" "My_Headers:5-pin_3,5mm_audio_jack_header" (id 2) (at 287.02 46.99 0)
       (effects (font (size 1.27 1.27)) hide)
     )
@@
       (effects (font (size 1.27 1.27)) hide)
     )
-    (property "Footprint" "" (id 2) (at 287.02 74.93 0)
+    (property "Footprint" "My_Headers:5-pin_3,5mm_audio_jack_header" (id 2) (at 287.02 74.93 0)
       (effects (font (size 1.27 1.27)) hide)
     )
@@
       (effects (font (size 1.27 1.27)) hide)
     )
-    (property "Footprint" "" (id 2) (at 279.4 123.19 0)
+    (property "Footprint" "My_Headers:4-pin_3_LED_header" (id 2) (at 279.4 123.19 0)
       (effects (font (size 1.27 1.27)) hide)
     )
@@
   (symbol_instances
     (path "/00000000-0000-0000-0000-00005e4000fe"
-      (reference "A1") (unit 1) (value "Arduino_UNO_R3") (footprint "My_Arduino:Arduino_UNO_R3_shield_large")
+      (reference "A1") (unit 1) (value "Arduino_UNO_R3") (footprint "Module:Arduino_UNO_R3")
     )
     (path "/14bec114-4374-48cb-ae22-cfdfe1c09b80"
@@
     )
     (path "/00000000-0000-0000-0000-00005e58ee76"
-      (reference "J6") (unit 1) (value "5-pin_3-pole_3,5mm_audio_header") (footprint "")
+      (reference "J6") (unit 1) (value "5-pin_3-pole_3,5mm_audio_header") (footprint "My_Headers:5-pin_3,5mm_audio_jack_header")
     )
     (path "/00000000-0000-0000-0000-00005e59be1a"
-      (reference "J7") (unit 1) (value "5-pin_3-pole_3,5mm_audio_header") (footprint "")
+      (reference "J7") (unit 1) (value "5-pin_3-pole_3,5mm_audio_header") (footprint "My_Headers:5-pin_3,5mm_audio_jack_header")
     )
     (path "/00000000-0000-0000-0000-00005e5a234b"
-      (reference "J8") (unit 1) (value "5-pin_3-pole_3,5mm_audio_header") (footprint "")
+      (reference "J8") (unit 1) (value "5-pin_3-pole_3,5mm_audio_header") (footprint "My_Headers:5-pin_3,5mm_audio_jack_header")
     )
     (path "/00000000-0000-0000-0000-00005e5abb60"
-      (reference "J9") (unit 1) (value "5-pin_3-pole_3,5mm_audio_header") (footprint "")
+      (reference "J9") (unit 1) (value "5-pin_3-pole_3,5mm_audio_header") (footprint "My_Headers:5-pin_3,5mm_audio_jack_header")
     )
     (path "/00000000-0000-0000-0000-00005e5ad60c"
-      (reference "J10") (unit 1) (value "5-pin_3-pole_3,5mm_audio_header") (footprint "")
+      (reference "J10") (unit 1) (value "5-pin_3-pole_3,5mm_audio_header") (footprint "My_Headers:5-pin_3,5mm_audio_jack_header")
     )
     (path "/2814365d-62f1-48f9-a546-1bbc5f4174c7"
-      (reference "J11") (unit 1) (value "4-pin_3LED_header") (footprint "")
+      (reference "J11") (unit 1) (value "4-pin_3LED_header") (footprint "My_Headers:4-pin_3_LED_header")
     )
     (path "/e5998ca8-a0c2-4b1d-8136-b090f3ae2262"
@@
     )
     (path "/00000000-0000-0000-0000-00005e54f8df"
-      (reference "U1") (unit 1) (value "DS18B20") (footprint "")
-    )
-  )
+      (reference "U1") (unit 1) (value "DS18B20") (footprint "Package_TO_SOT_THT:TO-92_Inline")
+    )
+  )
