File: KiCad/ardWeatherStation/ardWeatherStation.kicad_sch (KiCad schematic)
At the start: 14 parts, among them J3 16-pin_LCD_header

Commit message: schematics
Parts:
- A1: value (none) -> Arduino_UNO_R3
- D1: value (none) -> LED
- J1, J2: value (none) -> RJ45
- R1: value (none) -> 330R; footprint (none) -> My_Misc:R_Axial_DIN0207_L6.3mm_D2.5mm_P10.16mm_Horizontal_larger_pads
- R2, R3: value (none) -> 10k; footprint (none) -> My_Misc:R_Axial_DIN0207_L6.3mm_D2.5mm_P10.16mm_Horizontal_larger_pads
- R4: value (none) -> 15k; footprint (none) -> My_Misc:R_Axial_DIN0207_L6.3mm_D2.5mm_P10.16mm_Horizontal_larger_pads
- U1: value (none) -> Rain_bucket
- U2: value (none) -> Anemometer
- U3: value (none) -> Wind_vane
Changed lines of the file:
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@@
     (in_bom yes) (on_board yes)
     (property "Reference" "A1" (id 0) (at 224.79 63.9826 0))
-    (property "Value" "" (id 1) (at 224.79 66.294 0))
+    (property "Value" "Arduino_UNO_R3" (id 1) (at 224.79 66.294 0))
     (property "Footprint" "My_Arduino:Arduino_UNO_R3_shield_large" (id 2) (at 224.79 93.98 0)
       (effects (font (size 1.27 1.27) italic) hide)
@@
     (in_bom yes) (on_board yes)
     (property "Reference" "R3" (id 0) (at 166.37 76.0222 90))
-    (property "Value" "" (id 1) (at 166.37 78.3336 90))
-    (property "Footprint" "" (id 2) (at 166.37 79.502 90)
+    (property "Value" "10k" (id 1) (at 166.37 78.3336 90))
+    (property "Footprint" "My_Misc:R_Axial_DIN0207_L6.3mm_D2.5mm_P10.16mm_Horizontal_larger_pads" (id 2) (at 166.37 79.502 90)
       (effects (font (size 1.27 1.27)) hide)
     )
@@
     (in_bom yes) (on_board yes)
     (property "Reference" "R2" (id 0) (at 166.37 67.1322 90))
-    (property "Value" "" (id 1) (at 166.37 69.4436 90))
-    (property "Footprint" "" (id 2) (at 166.37 70.612 90)
+    (property "Value" "10k" (id 1) (at 166.37 69.4436 90))
+    (property "Footprint" "My_Misc:R_Axial_DIN0207_L6.3mm_D2.5mm_P10.16mm_Horizontal_larger_pads" (id 2) (at 166.37 70.612 90)
       (effects (font (size 1.27 1.27)) hide)
     )
@@
       (effects (font (size 1.27 1.27)) (justify right))
     )
-    (property "Value" "" (id 1) (at 62.992 93.6752 90)
+    (property "Value" "RJ45" (id 1) (at 62.992 93.6752 90)
       (effects (font (size 1.27 1.27)) (justify right))
     )
@@
     (in_bom yes) (on_board yes)
     (property "Reference" "D1" (id 0) (at 166.1922 40.2336 0))
-    (property "Value" "" (id 1) (at 166.1922 42.545 0))
+    (property "Value" "LED" (id 1) (at 166.1922 42.545 0))
     (property "Footprint" "My_Misc:LED_D5.0mm_large" (id 2) (at 166.37 45.72 0)
       (effects (font (size 1.27 1.27)) hide)
@@
     (in_bom yes) (on_board yes)
     (property "Reference" "R1" (id 0) (at 166.37 49.3522 90))
-    (property "Value" "" (id 1) (at 166.37 51.6636 90))
-    (property "Footprint" "" (id 2) (at 166.37 52.832 90)
+    (property "Value" "330R" (id 1) (at 166.37 51.6636 90))
+    (property "Footprint" "My_Misc:R_Axial_DIN0207_L6.3mm_D2.5mm_P10.16mm_Horizontal_larger_pads" (id 2) (at 166.37 52.832 90)
       (effects (font (size 1.27 1.27)) hide)
     )
@@
     (in_bom yes) (on_board yes)
     (property "Reference" "R4" (id 0) (at 261.62 91.2622 90))
-    (property "Value" "" (id 1) (at 261.62 93.5736 90))
-    (property "Footprint" "" (id 2) (at 261.62 94.742 90)
+    (property "Value" "15k" (id 1) (at 261.62 93.5736 90))
+    (property "Footprint" "My_Misc:R_Axial_DIN0207_L6.3mm_D2.5mm_P10.16mm_Horizontal_larger_pads" (id 2) (at 261.62 94.742 90)
       (effects (font (size 1.27 1.27)) hide)
     )
@@
       (effects (font (size 1.27 1.27)) (justify right))
     )
-    (property "Value" "" (id 1) (at 62.992 116.8908 90)
+    (property "Value" "RJ45" (id 1) (at 62.992 116.8908 90)
       (effects (font (size 1.27 1.27)) (justify right))
     )
@@
       (effects (font (size 1.27 1.27)) (justify right))
     )
-    (property "Value" "" (id 1) (at 128.9812 175.133 0)
+    (property "Value" "Wind_vane" (id 1) (at 128.9812 175.133 0)
       (effects (font (size 1.27 1.27)) (justify right))
     )
@@
       (effects (font (size 1.27 1.27)) (justify right))
     )
-    (property "Value" "" (id 1) (at 121.3612 151.003 0)
+    (property "Value" "Anemometer" (id 1) (at 121.3612 151.003 0)
       (effects (font (size 1.27 1.27)) (justify right))
     )
@@
       (effects (font (size 1.27 1.27)) (justify right))
     )
-    (property "Value" "" (id 1) (at 122.6312 130.683 0)
+    (property "Value" "Rain_bucket" (id 1) (at 122.6312 130.683 0)
       (effects (font (size 1.27 1.27)) (justify right))
     )
